Commit message: Fix kbot-v2-legs asset: hip_roll motor, root body name, foot sites
Asset fixes needed to make kbot-v2-legs train cleanly with ksim:

- hip_roll: was tagged as motor_03 (11 Nm); the hardware uses motor_04
  (22 Nm) like the knee.  Updated MJCF class, URDF effort/velocity
  limits, and metadata.json (actuator_type robstride_03 -> robstride_04,
  soft_torque_limit 42 -> 84 Nm).
- root body renamed floating_base_link -> base, required by the
  mujoco_scenes scene template's <light target="base"/>.
- Added heel and toe sites (left_foot_heel/toe, right_foot_heel/toe)
  inside each foot body so FeetEndpointsObservation can resolve them.

Verified: nu=10, nsite=8, mass=13.064 kg.

Co-Authored-By: Claude Opus 4.7 <noreply@anthropic.com>

File: gim_test/sim_assets/kbot-v2-legs/robot.urdf (robot description, URDF)
Before this commit: robot kbotv2p0_nohands, 13 links, 12 joints
Joints:
- removed joint dof_left_hip_roll_03
- removed joint dof_right_hip_roll_03
- added joint dof_left_hip_roll_04: type revolute, parent KC_D_102L_L_Hip_Yoke_Drive, child RS03_5, origin xyz=-0.028250 0.030000 -0.071000 rpy=0 1.570796 0, axis 0 0 -1, limit lower=-0.209440 upper=2.268928 effort=120 velocity=17.488
- added joint dof_right_hip_roll_04: type revolute, parent KC_D_102R_R_Hip_Yoke_Drive, child RS03_4, origin xyz=-0.028250 -0.030000 -0.071000 rpy=3.141593 -1.570796 0, axis 0 0 -1, limit lower=-2.268928 upper=0.209440 effort=120 velocity=17.488
